Commit message: v0.0.4 -fixed intertia bug in gripper -added claw -renamed files

File: pap_arm/urdf/gripper.xacro (robot description, xacro)
@@ -24,5 +24,5 @@
                 </geometry>
             </collision>
-            <xacro:box_inertia m="3.0" x="0.02" y="0.02" z="0.04" o_xyz="0 0 0" o_rpy="0 0 0"/>
+            <xacro:box_inertia m="3.0" x="${gripper_finger_length}" y="${gripper_finger_width}" z="${gripper_finger_height}" o_xyz="0 0 ${gripper_finger_height/2.0}" o_rpy="0 0 0"/>
         </link>
     </xacro:macro>

File: pap_arm/urdf/pap_arm.xacro (robot description, xacro)
@@ -4,9 +4,15 @@
     <xacro:include filename="$(find pap_arm)/urdf/pap_arm_links.xacro"/>
     <xacro:include filename="$(find pap_arm)/urdf/pap_arm_gazebo.xacro"/>
-    <xacro:include filename="$(find pap_arm)/urdf/gripper.xacro"/>
-    <joint name="end_effector_gripper" type="fixed">
+    <!-- <xacro:include filename="$(find pap_arm)/urdf/gripper.xacro"/> -->
+    <xacro:include filename="$(find pap_arm)/urdf/claw.xacro"/>
+    <!-- <joint name="end_effector_gripper" type="fixed">
         <origin xyz="0.0 0.0 ${gripper_base_height/2.0}" rpy="0.0 0.0 0.0"/>
         <parent link="end_effector"/>
         <child link="gripper_base"/>
+    </joint> -->
+    <joint name="end_effector_gripper" type="fixed">
+        <origin xyz="0.0 0.0 ${claw_base_length/2.0}" rpy="0.0 0.0 0.0"/>
+        <parent link="end_effector"/>
+        <child link="claw_base"/>
     </joint>
 </robot>
