Commit message: v0.0.5 -improved claw design -renamed gazebo bringup

File: pap_arm/urdf/claw.xacro (robot description, xacro)
@@ -10,7 +10,4 @@
     <!-- XACRO FOR CLAW FINGERS -->
     <xacro:macro name="claw_finger" params="name">
-        <!-- DUMMY OFFEST LINK -->
-        <link name="claw_finger_offset_${name}">
-        </link>
         <!-- FINGER LINK 1 -->
         <link name="${name}_claw_finger">
@@ -28,5 +25,5 @@
                 </geometry>
             </collision>
-            <xacro:box_inertia m="3.0" x="${claw_finger_length}" y="${claw_finger_width}" z="${claw_finger_height}" o_xyz="0 0 ${claw_finger_height/2.0}" o_rpy="0 0 0"/>
+            <xacro:box_inertia m="0.2" x="${claw_finger_length}" y="${claw_finger_width}" z="${claw_finger_height}" o_xyz="0 0 ${claw_finger_height/2.0}" o_rpy="0 0 0"/>
         </link>
         <!-- FINGER LINK 2 -->
@@ -45,13 +42,8 @@
                 </geometry>
             </collision>
-            <xacro:box_inertia m="3.0" x="${claw_finger_length}" y="${claw_finger_width}" z="${claw_finger_height}" o_xyz="0 0 ${claw_finger_height/2.0}" o_rpy="0 0 0"/>
+            <xacro:box_inertia m="0.1" x="${claw_finger_length}" y="${claw_finger_width}" z="${claw_finger_height}" o_xyz="0 0 ${claw_finger_height/2.0}" o_rpy="0 0 0"/>
         </link>
-        <joint name="offset_joint_${name}" type="fixed">
-            <origin xyz="${claw_finger_offset} 0 0" rpy="0 0.5 0"/>
-            <parent link="claw_finger_offset_${name}"/>
-            <child link="${name}_claw_finger"/>
-        </joint>
         <joint name="finger_claw_${name}" type="fixed">
-            <origin xyz="0 0 ${claw_finger_height}" rpy="0 -0.5 0"/>
+            <origin xyz="0 0 ${claw_finger_height}" rpy="0 0.5 0"/>
             <parent link="${name}_claw_finger"/>
             <child link="gripper_claw_${name}"/>
@@ -78,14 +70,14 @@
     <xacro:claw_finger name="three"/>
     <joint name="claw_base_finger_one" type="revolute">
-        <origin xyz="0 0.0 -${claw_base_length/1.5}" rpy="0.0 0.0 0.0"/>
+        <origin xyz="-${claw_finger_offset} 0.0 ${claw_base_length/2}" rpy="0.0 -0.5  0.0"/>
         <parent link="claw_base"/>
-        <child link="claw_finger_offset_one"/>
+        <child link="one_claw_finger"/>
         <axis xyz="0.0 1.0 0.0"/>
-        <limit lower="0" upper="-0.6" effort="0.0" velocity="0.0"/>
+        <limit lower="0" upper="0.75" effort="0.0" velocity="0.0"/>
     </joint>
     <joint name="claw_base_finger_two" type="revolute">
-        <origin xyz="0 0.0 -${claw_base_length/1.5}" rpy="0.0  0.0 2.05"/>
+        <origin xyz="${claw_finger_offset*0.5} ${0.866*claw_finger_offset} ${claw_base_length/2}" rpy="0.0  -0.5 -2.09"/>
         <parent link="claw_base"/>
-        <child link="claw_finger_offset_two"/>
+        <child link="two_claw_finger"/>
         <axis xyz="0.0 1.0 0.0"/>
         <limit lower="0.0" upper="1.2" effort="0.0" velocity="0.0"/>
@@ -93,7 +85,7 @@
     </joint>
     <joint name="claw_base_finger_three" type="revolute">
-        <origin xyz="0 0.0 -${claw_base_length/1.5}" rpy="0.0  0.0 4.10"/>
+        <origin xyz="${claw_finger_offset*0.5} ${-0.866*claw_finger_offset} ${claw_base_length/2}" rpy="0.0 -0.5 2.09"/>
         <parent link="claw_base"/>
-        <child link="claw_finger_offset_three"/>
+        <child link="three_claw_finger"/>
         <axis xyz="0.0 1.0 0.0"/>
         <limit lower="0.0" upper="1.2" effort="0.0" velocity="0.0"/>

Commit message: v0.0.6 -fixed claw -added in moveitconfig -setup for moveitconfig

File: pap_arm/urdf/claw.xacro (robot description, xacro)
@@ -8,5 +8,5 @@
     <xacro:property name="claw_finger_height" value="0.04"/>
     <xacro:property name="claw_finger_offset" value="0.05"/>
-    <!-- XACRO FOR CLAW FINGERS -->
+    <!-- XACRO FOR CLAWS -->
     <xacro:macro name="claw_finger" params="name">
         <!-- FINGER LINK 1 -->
@@ -25,5 +25,5 @@
                 </geometry>
             </collision>
-            <xacro:box_inertia m="0.2" x="${claw_finger_length}" y="${claw_finger_width}" z="${claw_finger_height}" o_xyz="0 0 ${claw_finger_height/2.0}" o_rpy="0 0 0"/>
+<!--             <xacro:box_inertia m="0.2" x="${claw_finger_length}" y="${claw_finger_width}" z="${claw_finger_height}" o_xyz="0 0 ${claw_finger_height/2.0}" o_rpy="0 0 0"/> -->
         </link>
         <!-- FINGER LINK 2 -->
@@ -42,8 +42,8 @@
                 </geometry>
             </collision>
-            <xacro:box_inertia m="0.1" x="${claw_finger_length}" y="${claw_finger_width}" z="${claw_finger_height}" o_xyz="0 0 ${claw_finger_height/2.0}" o_rpy="0 0 0"/>
+<!--             <xacro:box_inertia m="0.1" x="${claw_finger_length}" y="${claw_finger_width}" z="${claw_finger_height}" o_xyz="0 0 ${claw_finger_height/2.0}" o_rpy="0 0 0"/> -->
         </link>
         <joint name="finger_claw_${name}" type="fixed">
-            <origin xyz="0 0 ${claw_finger_height}" rpy="0 0.5 0"/>
+            <origin xyz="0 0 ${claw_finger_height*1.1}" rpy="0 0.5 0"/>
             <parent link="${name}_claw_finger"/>
             <child link="gripper_claw_${name}"/>
@@ -51,6 +51,6 @@
     </xacro:macro>
     <link name="claw_base">
-        <xacro:box_inertia m="3.0" x="${2*claw_base_radius}"  y="${2*claw_base_radius}"  z="${claw_base_length}"  o_xyz="0 0 0" o_rpy="0 0 0"/>
-        <visual name="">
+<!--         <xacro:box_inertia m="3.0" x="${2*claw_base_radius}"  y="${2*claw_base_radius}"  z="${claw_base_length}"  o_xyz="0 0 0" o_rpy="0 0 0"/> -->
+        <visual >
             <origin xyz="0.0 0.0 0.0" rpy="0.0 0.0 0.0"/>
             <geometry>
@@ -70,24 +70,24 @@
     <xacro:claw_finger name="three"/>
     <joint name="claw_base_finger_one" type="revolute">
-        <origin xyz="-${claw_finger_offset} 0.0 ${claw_base_length/2}" rpy="0.0 -0.5  0.0"/>
+        <origin xyz="-${claw_finger_offset} 0.0 ${claw_base_length/1.5}" rpy="0.0 -0.5  0.0"/>
         <parent link="claw_base"/>
         <child link="one_claw_finger"/>
         <axis xyz="0.0 1.0 0.0"/>
-        <limit lower="0" upper="0.75" effort="0.0" velocity="0.0"/>
+        <limit lower="0" upper="0.75" effort="10.0" velocity="10.0"/>
     </joint>
     <joint name="claw_base_finger_two" type="revolute">
-        <origin xyz="${claw_finger_offset*0.5} ${0.866*claw_finger_offset} ${claw_base_length/2}" rpy="0.0  -0.5 -2.09"/>
+        <origin xyz="${claw_finger_offset*0.5} ${0.866*claw_finger_offset} ${claw_base_length/1.5}" rpy="0.0  -0.5 -2.09"/>
         <parent link="claw_base"/>
         <child link="two_claw_finger"/>
         <axis xyz="0.0 1.0 0.0"/>
-        <limit lower="0.0" upper="1.2" effort="0.0" velocity="0.0"/>
+        <limit lower="0.0" upper="1.2" effort="10.0" velocity="10.0"/>
         <mimic joint="claw_base_finger_one" multiplier="1.0"/>
     </joint>
     <joint name="claw_base_finger_three" type="revolute">
-        <origin xyz="${claw_finger_offset*0.5} ${-0.866*claw_finger_offset} ${claw_base_length/2}" rpy="0.0 -0.5 2.09"/>
+        <origin xyz="${claw_finger_offset*0.5} ${-0.866*claw_finger_offset} ${claw_base_length/1.5}" rpy="0.0 -0.5 2.09"/>
         <parent link="claw_base"/>
         <child link="three_claw_finger"/>
         <axis xyz="0.0 1.0 0.0"/>
-        <limit lower="0.0" upper="1.2" effort="0.0" velocity="0.0"/>
+        <limit lower="0.0" upper="1.2" effort="10.0" velocity="10.0"/>
         <mimic joint="claw_base_finger_one" multiplier="1.0"/>
     </joint>

File: pap_arm/urdf/gripper.xacro (robot description, xacro)
@@ -24,10 +24,11 @@
                 </geometry>
             </collision>
-            <xacro:box_inertia m="3.0" x="${gripper_finger_length}" y="${gripper_finger_width}" z="${gripper_finger_height}" o_xyz="0 0 ${gripper_finger_height/2.0}" o_rpy="0 0 0"/>
+<!--             <xacro:box_inertia m="3.0" x="${gripper_finger_length}" y="${gripper_finger_width}" z="${gripper_finger_height}" o_xyz="0 0 ${gripper_finger_height/2.0}" o_rpy="0 0 0"/>
+ -->
         </link>
     </xacro:macro>
     <link name="gripper_base">
-        <xacro:box_inertia m="3.0" x="${gripper_base_length}" y="${gripper_base_width}" z="${gripper_base_height}" o_xyz="0 0 0" o_rpy="0 0 0"/>
-        <visual name="">
+<!--         <xacro:box_inertia m="3.0" x="${gripper_base_length}" y="${gripper_base_width}" z="${gripper_base_height}" o_xyz="0 0 0" o_rpy="0 0 0"/>
+ -->        <visual name="">
             <origin xyz="0.0 0.0 0.0" rpy="0.0 0.0 0.0"/>
             <geometry>

File: pap_arm/urdf/pap_arm.xacro (robot description, xacro)
@@ -6,4 +6,5 @@
     <!-- <xacro:include filename="$(find pap_arm)/urdf/gripper.xacro"/> -->
     <xacro:include filename="$(find pap_arm)/urdf/claw.xacro"/>
+    <xacro:include filename="$(find pap_arm)/urdf/pap_arm.ros2_control.xacro"/>
     <!-- <joint name="end_effector_gripper" type="fixed">
         <origin xyz="0.0 0.0 ${gripper_base_height/2.0}" rpy="0.0 0.0 0.0"/>

File: pap_arm/urdf/pap_arm_links.xacro (robot description, xacro)
@@ -19,5 +19,5 @@
     <xacro:property name="end_effector_radius" value="0.02"/>
     <!-- LINKS -->
-    <link name="base_footprint"></link>
+<!--     <link name="base_footprint"></link> -->
     <link name="base_link">
         <visual>
@@ -28,5 +28,5 @@
             <material name="grey"/>
         </visual>
-        <xacro:box_inertia m="3.0" x="${base_length}" y="${base_width}" z="${base_height}" o_xyz="0 0 0" o_rpy="0 0 0"/>
+<!--         <xacro:box_inertia m="3.0" x="${base_length}" y="${base_width}" z="${base_height}" o_xyz="0 0 0" o_rpy="0 0 0"/> -->
         <collision>
             <geometry>
@@ -45,5 +45,5 @@
                 <material name="${color}"/>
             </visual>
-            <xacro:box_inertia m="${mass}" x="${radius*2.0}" y="${radius*2.0}" z="${length}" o_xyz="0 0 ${length/2}" o_rpy="0 0 0"/>
+<!--             <xacro:box_inertia m="${mass}" x="${radius*2.0}" y="${radius*2.0}" z="${length}" o_xyz="0 0 ${length/2}" o_rpy="0 0 0"/> -->
             <collision>
                 <geometry>
@@ -61,25 +61,11 @@
     <xacro:cylindrical_link name="link6" length="${link6_length}" radius="${link6_radius}" mass="0.2" color="blue"/>
     <link name="end_effector">
-        <!-- <visual>
-            <geometry>
-                <sphere radius="${end_effector_radius}"/>
-            </geometry>
-            <origin xyz="0 0 0" rpy="0 0 0"/>
-            <material name="blue"/>
-        </visual>
-        <xacro:solid_sphere_inertia m="0.1" r="${end_effector_radius}" o_xyz="0 0 0" o_rpy="0 0 0"/>
-        <collision>
-            <geometry>
-                <sphere radius="${end_effector_radius}"/>
-            </geometry>
-            <origin xyz="0 0 0" rpy="0 0 0"/>
-        </collision>     -->
     </link>
     <!-- JOINTS -->
-    <joint name="base_footprint_base" type="fixed">
+    <!-- <joint name="base_footprint_base" type="fixed">
         <parent link="base_footprint"/>
         <child link="base_link"/>
         <origin xyz="0 0 ${base_height/2.0}" rpy="0 0 0"/>
-    </joint>
+    </joint> -->
     <joint name="base_link_link1" type="revolute">
         <parent link="base_link"/>
