Commit message: bleh

File: panda_description/urdf/gazebo.xacro (robot description, xacro)
@@ -2,23 +2,8 @@
 <robot xmlns:xacro="http://www.ros.org/wiki/xacro" name="panda">
   <!-- ROS 2 Control -->
-  <!-- ROS 2 Humble -->
   <gazebo>
-    <xacro:if value="$(arg is_ignition)">
-      <plugin filename="ign_ros2_control-system" name="ign_ros2_control::IgnitionROS2ControlPlugin">
-        <parameters>$(find panda_controller)/config/panda_controllers.yaml</parameters>
-      </plugin>
-      <plugin filename="ignition-gazebo-sensors-system" name="ignition::gazebo::systems::Sensors">
-        <render_engine>ogre2</render_engine>
-      </plugin>
-    </xacro:if>
-    <!-- ROS 2 Iron or above -->
-    <xacro:unless value="$(arg is_ignition)">
-      <plugin filename="gz_ros2_control-system" name="gz_ros2_control::GazeboSimROS2ControlPlugin">
-        <parameters>$(find panda_controller)/config/panda_controllers.yaml</parameters>
-      </plugin>
-      <plugin filename="gz-sim-sensors-system" name="gz::sim::systems::Sensors">
-        <render_engine>ogre2</render_engine>
-      </plugin>
-    </xacro:unless>
+    <plugin filename="libgz_ros2_control-system.so" name="gz_ros2_control::GazeboSimROS2ControlPlugin">
+      <parameters>$(find panda_controller)/config/ros2_controllers.yaml</parameters>
+    </plugin>
   </gazebo>
 </robot>

File: panda_description/urdf/panda.urdf.xacro (robot description, xacro)
@@ -2,8 +2,8 @@
 <robot name="panda" xmlns:xacro="http://www.ros.org/wiki/xacro">
   <xacro:arg name="is_ignition" default="false"/>
+  <xacro:include filename="$(find panda_description)/urdf/common_properties.urdf.xacro" />
+  <xacro:include filename="$(find panda_description)/urdf/arm.xacro" />
+<!--   <xacro:include filename="$(find panda_description)/urdf/sensors.xacro" />-->
+  <xacro:include filename="$(find panda_description)/urdf/gazebo.xacro" />
   <xacro:include filename="$(find panda_description)/urdf/panda.ros2_control.xacro" />
-  <xacro:include filename="$(find panda_description)/urdf/arm.xacro" />
-<!--   <xacro:include filename="$(find panda_description)/urdf/sensors.xacro" />
-  <xacro:include filename="$(find panda_description)/urdf/gazebo.xacro" />
-  <xacro:include filename="$(find panda_description)/urdf/ros2control.xacro" />-->
 </robot>

File: panda_description/urdf/panda_.ros2_control.xacro (robot description, xacro)
@@ -1,19 +1,9 @@
 <?xml version="1.0"?>
-<robot xmlns:xacro="http://www.ros.org/wiki/xacro" name="panda">
+<robot xmlns:xacro="http://www.ros.org/wiki/xacro" >
   <xacro:property name="PI" value="3.14159265359" />
-  <ros2_control name="RobotSystem" type="system">
-    <!-- ros2_control Gazebo -->
-    <!-- ROS 2 Humble -->
-    <xacro:if value="$(arg is_ignition)">
-      <hardware>
-        <plugin>ign_ros2_control/IgnitionSystem</plugin>
-      </hardware>
-    </xacro:if>
-    <!-- ROS 2 Iron or above -->
-    <xacro:unless value="$(arg is_ignition)">
-      <hardware>
-        <plugin>gz_ros2_control/GazeboSimSystem</plugin>
-      </hardware>
-    </xacro:unless>
+  <ros2_control name="GazeboSimSystem" type="system">
+    <hardware>
+      <plugin>gz_ros2_control/GazeboSimSystem</plugin>
+    </hardware>
     <!-- Joint 1 -->
     <joint name="panda_joint1">
@@ -22,5 +12,7 @@
         <param name="max">2.9671</param>
       </command_interface>
-      <state_interface name="position"/>
+      <state_interface name="position">
+        <param name="initial_value">0</param>
+      </state_interface>
     </joint>
     <!-- Joint 2 -->
@@ -30,5 +22,7 @@
         <param name="max">1.8326</param>
       </command_interface>
-      <state_interface name="position"/>
+      <state_interface name="position">
+        <param name="initial_value">0</param>
+      </state_interface>
     </joint>
     <!-- Joint 3 -->
@@ -38,5 +32,7 @@
         <param name="max">2.9671</param>
       </command_interface>
-      <state_interface name="position"/>
+      <state_interface name="position">
+        <param name="initial_value">0</param>
+      </state_interface>
     </joint>
     <!-- Joint 4 -->
@@ -46,5 +42,7 @@
         <param name="max">0.0</param>
       </command_interface>
-      <state_interface name="position"/>
+      <state_interface name="position">
+        <param name="initial_value">0</param>
+      </state_interface>
     </joint>
     <!-- Joint 5 -->
@@ -54,5 +52,7 @@
         <param name="max">2.9671</param>
       </command_interface>
-      <state_interface name="position"/>
+      <state_interface name="position">
+        <param name="initial_value">0</param>
+      </state_interface>
     </joint>
     <!-- Joint 6 -->
@@ -62,5 +62,7 @@
         <param name="max">3.8223</param>
       </command_interface>
-      <state_interface name="position"/>
+      <state_interface name="position">
+        <param name="initial_value">0</param>
+      </state_interface>
     </joint>
     <!-- Joint 7 -->
@@ -70,5 +72,7 @@
         <param name="max">2.9671</param>
       </command_interface>
-      <state_interface name="position"/>
+      <state_interface name="position">
+        <param name="initial_value">0</param>
+      </state_interface>
     </joint>
     <!-- Gripper Finger Joint 1 -->
@@ -78,5 +82,7 @@
         <param name="max">0.04</param>
       </command_interface>
-      <state_interface name="position"/>
+      <state_interface name="position">
+        <param name="initial_value">0</param>
+      </state_interface>
     </joint>
     <!-- Gripper Finger Joint 2 (Mimics Joint 1) -->
@@ -86,5 +92,7 @@
         <param name="max">0.04</param>
       </command_interface>
-      <state_interface name="position"/>
+      <state_interface name="position">
+        <param name="initial_value">0</param>
+      </state_interface>
     </joint>
   </ros2_control>

File: panda_moveit_config/config/panda.ros2_control.xacro (robot description, xacro)
@@ -2,5 +2,5 @@
 <robot xmlns:xacro="http://www.ros.org/wiki/xacro">
     <xacro:macro name="panda_ros2_control" params="name initial_positions_file">
-        <xacro:property name="initial_positions" value="${load_yaml(initial_positions_file)['initial_positions']}"/>
+        <xacro:property name="initial_positions" value="${xacro.load_yaml(initial_positions_file)['initial_positions']}"/>
         <ros2_control name="${name}" type="system">
             <hardware>
