Commit message: v0.1.6 Updating moveit_commander -simulation.launch.xml:added commander node -arm.xacro:updated joint4 limits to match soft limits -my_robot_commander/src: renamed base_link with panda_link0 to match new URDF

File: panda_description/urdf/arm.xacro (robot description, xacro)
@@ -133,5 +133,5 @@
     <child link="panda_link4"/>
     <axis xyz="0 0 1"/>
-    <limit effort="30.0" lower="-3.1416" upper="0.0" velocity="10.0"/>
+    <limit effort="30.0" lower="-3.1416" upper="0.0698" velocity="10.0"/>
   </joint>
   <!-- Link 5 -->

Commit message: v0.1.7-b Fixing CV Pipeline -gazebo_bridge.yaml:added brige for camera_info gz topic -arm.xacro:added test link to confirm dist. from panda_link7 to gripper -panda_ros2_control.xacro:  changed initial values to avoid collisions -color_detector.py: corrected camera specs,coordinate calc, Z adjus

File: panda_description/urdf/arm.xacro (robot description, xacro)
@@ -234,4 +234,10 @@
       </inertial>
   </link>
+  <link name="test_link"/>
+  <joint name="joint_name" type="fixed">
+    <parent link="panda_link7"/>
+    <child link="test_link"/>
+    <origin rpy="0 0 0" xyz="0 0 0.21"/>
+  </joint>
   <!-- Hand Joint -->
   <joint name="panda_hand_joint" type="fixed">

File: panda_description/urdf/panda_.ros2_control.xacro (robot description, xacro)
@@ -64,5 +64,5 @@
       </command_interface>
       <state_interface name="position">
-        <param name="initial_value">0</param>
+        <param name="initial_value">0.785</param>
       </state_interface>
     </joint>
@@ -84,5 +84,5 @@
       </command_interface>
       <state_interface name="position">
-        <param name="initial_value">0</param>
+        <param name="initial_value">0.01</param>
       </state_interface>
     </joint>
@@ -94,5 +94,5 @@
       </command_interface>
       <state_interface name="position">
-        <param name="initial_value">0</param>
+        <param name="initial_value">0.01</param>
       </state_interface>
     </joint>

Commit message: v0.1.8 Integrating tool_center_link -arm.xacro:rename test_link -> tool_center_link; joint_name->tool_center -deleted duplicate ros2_controllers.yaml from bringup -moveit_launch,gazebo.xacro,panda_ros2_control: change file path -panda.srdf: added tool_center to arm group -color_detector.py: Z fixed to only comp for block height

File: panda_description/urdf/arm.xacro (robot description, xacro)
@@ -234,8 +234,8 @@
       </inertial>
   </link>
-  <link name="test_link"/>
-  <joint name="joint_name" type="fixed">
+  <link name="tool_center_link"/>
+  <joint name="tool_center" type="fixed">
     <parent link="panda_link7"/>
-    <child link="test_link"/>
+    <child link="tool_center_link"/>
     <origin rpy="0 0 0" xyz="0 0 0.21"/>
   </joint>

File: panda_description/urdf/gazebo.xacro (robot description, xacro)
@@ -4,5 +4,5 @@
   <gazebo>
     <plugin filename="libgz_ros2_control-system.so" name="gz_ros2_control::GazeboSimROS2ControlPlugin">
-      <parameters>$(find panda_bringup)/config/ros2_controllers.yaml</parameters>
+      <parameters>$(find panda_moveit_config)/config/ros2_controllers.yaml</parameters>
     </plugin>
   </gazebo>

File: panda_description/urdf/panda_.ros2_control.xacro (robot description, xacro)
@@ -5,5 +5,5 @@
     <hardware>
       <plugin>gz_ros2_control/GazeboSimSystem</plugin>
-        <parameters>$(find panda_bringup)/config/ros2_controllers.yaml</parameters>
+        <parameters>$(find panda_moveit_config)/config/ros2_controllers.yaml</parameters>
     </hardware>
     <!-- Joint 1 -->

Commit message: v0.1.8 Implementing Pick and Place -added cv_pick_and_place node -added ColorCoordinates custom message -added both files to respective CmakeLists -gazebo_launch.xml: using test_world_2, added use_sim_time=true params -simulation.launch.xml: added cv_pick_and_place node to launch -added test_world_2: new test world with diff block arrangement -arm.xacro: increased finger upper limit -panda_.ros2_control.xacro: increased  gripper finger upper limit; changed init value to non zero cause of startstaterror -moveit_controllers.yaml: added trajectory execution params -moveit.rviz -panda.srdf:modified some poses -color_detector.py: integrated custom msg; flipped camera Z axis; fixed height comp

File: panda_description/urdf/arm.xacro (robot description, xacro)
@@ -284,4 +284,6 @@
       </inertial>
   </link>
+<!-- UPPER JOINT LIMITS HAVE BEEN SET TO 0.15(3x the effective upper limit of 0.05) to cricumvent an error where
+      the gripper would tilt one side causing start state to be out of bounds-->
   <!-- Finger Joint 1 -->
   <joint name="panda_finger_joint1" type="prismatic">
@@ -290,5 +292,5 @@
     <origin rpy="0 0 0" xyz="0 0 0.0584"/>
     <axis xyz="0 1 0"/>
-    <limit effort="30.0" lower="0.0" upper="0.04" velocity="10.0"/>
+    <limit effort="30.0" lower="0.0" upper="0.15" velocity="10.0"/>
   </joint>
   <!-- Finger Joint 2 -->
@@ -298,5 +300,5 @@
     <origin rpy="0 0 0" xyz="0 0 0.0584"/>
     <axis xyz="0 -1 0"/>
-    <limit effort="30.0" lower="0.0" upper="0.04" velocity="10.0"/>
+    <limit effort="30.0" lower="0.0" upper="0.15" velocity="10.0"/>
     <!-- <mimic joint="panda_finger_joint1" multiplier="-1"/> -->
   </joint>

File: panda_description/urdf/panda_.ros2_control.xacro (robot description, xacro)
@@ -81,8 +81,8 @@
       <command_interface name="position">
         <param name="min">0.0</param>
-        <param name="max">0.04</param>
+        <param name="max">0.05</param>
       </command_interface>
       <state_interface name="position">
-        <param name="initial_value">0.01</param>
+        <param name="initial_value">0.001</param>
       </state_interface>
     </joint>
@@ -91,8 +91,8 @@
       <command_interface name="position">
         <param name="min">0.0</param>
-        <param name="max">0.04</param>
+        <param name="max">0.05</param>
       </command_interface>
       <state_interface name="position">
-        <param name="initial_value">0.01</param>
+        <param name="initial_value">0.001</param>
       </state_interface>
     </joint>
